Commit message: update

File: fwdis/urdf/base/base.urdf.xacro (robot description, xacro)
@@ -1,5 +1,5 @@
 <?xml version="1.0"?>
 <robot xmlns:xacro="http://ros.org/wiki/xacro">
-  <xacro:include filename="$(find four_wheel_drive_independent_steering)/urdf/common.xacro"/>
+  <xacro:include filename="$(find fwdis)/urdf/common.xacro"/>
   <xacro:macro name="base" params="parent *joint_origin">
     <joint name="base_link_joint" type="fixed">
@@ -12,5 +12,5 @@
         <origin xyz="0 0 0" rpy="${M_PI/2} 0 ${M_PI/2}"/>
         <geometry>
-          <mesh filename="package://four_wheel_drive_independent_steering/meshes/STL/base2.stl" scale="0.001 0.001 0.001"/>
+          <mesh filename="package://fwdis/meshes/STL/base2.stl" scale="0.001 0.001 0.001"/>
         </geometry>
       </visual>
@@ -18,5 +18,5 @@
         <origin xyz="0 0 0" rpy="${M_PI/2} 0 ${M_PI/2}"/>
         <geometry>
-          <mesh filename="package://four_wheel_drive_independent_steering/meshes/STL/base2.stl" scale="0.001 0.001 0.001"/>
+          <mesh filename="package://fwdis/meshes/STL/base2.stl" scale="0.001 0.001 0.001"/>
         </geometry>
       </collision>

File: fwdis/urdf/building/building_simple.urdf.xacro (robot description, xacro)
@@ -2,5 +2,5 @@
 <robot name="building_simple" xmlns:xacro="http://ros.org/wiki/xacro">
   <static>true</static>
-  <xacro:include filename="$(find four_wheel_drive_independent_steering)/urdf/common.xacro"/>
+  <xacro:include filename="$(find fwdis)/urdf/common.xacro"/>
   <xacro:macro name="building">
     <link name="building">
@@ -8,5 +8,5 @@
         <origin xyz="-5 -5 0" rpy="${M_PI/2} 0 0"/>
         <geometry>
-          <mesh filename="package://four_wheel_drive_independent_steering/meshes/STL/building_simple.stl" scale="0.001 0.001 0.001"/>
+          <mesh filename="package://fwdis/meshes/STL/building_simple.stl" scale="0.001 0.001 0.001"/>
         </geometry>
         <material name="blue">
@@ -17,5 +17,5 @@
         <origin xyz="-5 -5 0" rpy="${M_PI/2} 0 0"/>
         <geometry>
-          <mesh filename="package://four_wheel_drive_independent_steering/meshes/STL/building_simple.stl" scale="0.001 0.001 0.001"/>
+          <mesh filename="package://fwdis/meshes/STL/building_simple.stl" scale="0.001 0.001 0.001"/>
         </geometry>
       </collision>

File: fwdis/urdf/sensors/lrf.urdf.xacro (robot description, xacro)
@@ -1,5 +1,5 @@
 <?xml version="1.0"?>
 <robot xmlns:xacro="http://ros.org/wiki/xacro">
-  <xacro:include filename="$(find four_wheel_drive_independent_steering)/urdf/common.xacro"/>
+  <xacro:include filename="$(find fwdis)/urdf/common.xacro"/>
   <xacro:macro name="hokuyo" params="prefix parent *joint_origin">
   <joint name="lrf_joint" type="fixed">
@@ -11,10 +11,10 @@
     <visual>
       <geometry>
-        <mesh filename="package://four_wheel_drive_independent_steering/meshes/STL/lrf.stl"/>
+        <mesh filename="package://fwdis/meshes/STL/lrf.stl"/>
       </geometry>
     </visual>
     <collision>
       <geometry>
-        <mesh filename="package://four_wheel_drive_independent_steering/meshes/STL/lrf.stl"/>
+        <mesh filename="package://fwdis/meshes/STL/lrf.stl"/>
       </geometry>
     </collision>

File: fwdis/urdf/steering/steering.urdf.xacro (robot description, xacro)
@@ -1,5 +1,5 @@
 <?xml version="1.0"?>
 <robot xmlns:xacro="http://ros.org/wiki/xacro">
-  <xacro:include filename="$(find four_wheel_drive_independent_steering)/urdf/common.xacro"/>
+  <xacro:include filename="$(find fwdis)/urdf/common.xacro"/>
   <property name="steering_radius" value="0.100"/>
   <property name="steering_width" value="0.100"/>
@@ -17,5 +17,5 @@
         <origin xyz="0 0 0" rpy="${M_PI/2} 0 ${M_PI/2}"/>
         <geometry>
-          <mesh filename="package://four_wheel_drive_independent_steering/meshes/STL/steering.stl" scale="0.001 0.001 0.001"/>
+          <mesh filename="package://fwdis/meshes/STL/steering.stl" scale="0.001 0.001 0.001"/>
         </geometry>
       </visual>

File: fwdis/urdf/wheel/wheel.urdf.xacro (robot description, xacro)
@@ -1,5 +1,5 @@
 <?xml version="1.0"?>
 <robot xmlns:xacro="http://ros.org/wiki/xacro">
-  <xacro:include filename="$(find four_wheel_drive_independent_steering)/urdf/common.xacro"/>
+  <xacro:include filename="$(find fwdis)/urdf/common.xacro"/>
   <property name="wheel_radius" value="0.100"/>
   <property name="wheel_width" value="0.030"/>
@@ -17,5 +17,5 @@
         <origin xyz="0 0.013208 0" rpy="${M_PI/2} 0 ${M_PI/2}"/>
         <geometry>
-          <mesh filename="package://four_wheel_drive_independent_steering/meshes/STL/wheel2.stl" scale="0.001 0.001 0.001"/>
+          <mesh filename="package://fwdis/meshes/STL/wheel2.stl" scale="0.001 0.001 0.001"/>
         </geometry>
       </visual>
